File: case/bottom_plate/yetis_bottom.kicad_pcb (KiCad board)
At the start: 2 copper layers, 146.3 x 134.6 mm, 7 parts

Commit message: Rename to yetiS
Signed-off-by: Norbert Pocs <norbertpocs0@gmail.com>
Other:
- board text added: "yetiS"
- board text removed: "yeti"
Changed lines of the file:
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@@
   (gr_line (start 211.074 87.884) (end 211.074 107.696)
     (stroke (width 0.1) (type default)) (layer "Edge.Cuts"))
-  (gr_text "yeti" (at 208.407 105.41) (layer "B.SilkS")
-    (effects (font (size 5 5) (thickness 1) bold) (justify left bottom mirror))
+  (gr_text "yetiS" (at 208.915 105.41) (layer "B.SilkS")
+    (effects (font (size 4.5 4.5) (thickness 1) bold) (justify left bottom mirror))
   )
-  (gr_text "yeti" (at 165.227 33.274 180) (layer "F.SilkS")
-    (effects (font (size 5 5) (thickness 1) bold) (justify left bottom))
+  (gr_text "yetiS" (at 166.37 33.274 180) (layer "F.SilkS")
+    (effects (font (size 4.5 4.5) (thickness 1) bold) (justify left bottom))
   )
 )
